File: VAR-PBB_v02/VAR-PBB_v02.sch (EAGLE design)
At the start: 32 parts, among them J1 ANDERSON_POWER_POLE, J11 CON1X2_SHROUDED, J2 ANDERSON_POWER_POLE, J3 CON1X2_SHROUDED, J4 CON1X2_SHROUDED, J5 CON1X2_SHROUDED, J6 CON1X2_SHROUDED, J7 CON1X2_SHROUDED, J8 CON1X2_SHROUDED, U1 OKI-78SR, U2 XL6009, U3 XL6009, U4 XL6009, U5 LP2985AIM5-1.5, U6 TPS259271DRCR

Commit message: Fixed misspelled top silk text "Engineering" to create v2.0 design.
Other:
- note added: "Release Notes: 01/30/2020 v1.0 - First version 10/31/2020 v2.0 - Fixed top silk screen misspelling of Engineering"
- note added: "VAR_PBB v02 Variable Power Board"
- note removed: "VAR_PBB v01 Variable Power Board"
Changed lines of the file:
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@@
 <?xml version="1.0" encoding="utf-8"?>
 <!DOCTYPE eagle SYSTEM "eagle.dtd">
-<eagle version="9.5.2">
+<eagle version="9.6.2">
 <drawing>
 <settings>
@@
 by Brian Schmalz of Schmalz Haus LLC</text>
 <text x="327.66" y="25.4" size="1.778" layer="98">Copyright 2020 Engineering^3 LLC</text>
-<text x="12.7" y="264.16" size="5.08" layer="98">VAR_PBB v01 Variable Power Board</text>
+<text x="12.7" y="264.16" size="5.08" layer="98">VAR_PBB v02 Variable Power Board</text>
 <text x="45.72" y="238.76" size="1.778" layer="98">Power Switch</text>
 <text x="196.596" y="232.918" size="1.778" layer="98">Power LED will turn off if any
@@
 <text x="199.644" y="207.772" size="1.778" layer="98">&gt;30V</text>
 <text x="72.39" y="205.232" size="1.778" layer="98">&gt;30V</text>
+<text x="12.7" y="160.02" size="1.778" layer="98">Release Notes:
+01/30/2020 v1.0 - First version
+10/31/2020 v2.0 - Fixed top silk screen misspelling of Engineering</text>
 </plain>
 <instances>
